File: GatorGrid-Kicad/Design V1.0/Design_V1.0.kicad_sch (KiCad schematic)
At the start: 16 parts, among them J1 Battery-Connector, SW1 SW_SPST, U1 TP4056

Commit message: updating KICAD
Connections:
- net VBUS: now also R2.1
- net STDBY: no longer names the net of U1.6 (~{STDBY})
- net STDBY: no longer R2.1
- no-connect marks 56 -> 57

Commit message: fixing KICAD
Connections:
- net GND: now also U1.1 (TEMP)
- no-connect marks 57 -> 56
Changed lines of the file:
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@@
-	)
-	(no_connect
-		(at 223.52 99.06)
 	)
 	(no_connect
@@
 					(unit 1)
 				)
+			)
+		)
+	)
+	(symbol
+		(lib_id "power:GND")
+		(at 223.52 99.06 270)
+		(unit 1)
+		(exclude_from_sim no)
+		(in_bom yes)
+		(on_board yes)
+		(dnp no)
+		(fields_autoplaced yes)
+		(property "Reference" "#PWR014"
+			(at 217.17 99.06 0)
+			(effects
+				(font
+					(size 1.27 1.27)
+				)
+				(hide yes)
+			)
+		)
+		(property "Value" "GND"
+			(at 219.71 99.0599 90)
+			(effects
+				(font
+					(size 1.27 1.27)
+				)
+				(justify right)
+			)
+		)
+		(property "Footprint" ""
+			(at 223.52 99.06 0)
+			(effects
+				(font
+					(size 1.27 1.27)
+				)
+				(hide yes)
+			)
+		)
+		(property "Datasheet" ""
+			(at 223.52 99.06 0)
+			(effects
+				(font
+					(size 1.27 1.27)
+				)
+				(hide yes)
+			)
+		)
+		(property "Description" "Power symbol creates a global label with name \"GND\" , ground"
+			(at 223.52 99.06 0)
+			(effects
+				(font
+					(size 1.27 1.27)
+				)
+				(hide yes)
+			)
+		)
+		(pin "1"
+		)
+		(instances
+			(project "Design_V1.0"
+				(path "/f525c831-642c-4dc1-b21c-e72cef05bbe4"
+					(reference "#PWR014")
+					(unit 1)
+				)
